Commit message: Added gazebo ros2 control plugin

File: xacro/rb1_ros2_base.urdf.xacro (robot description, xacro)
@@ -84,5 +84,35 @@
 		<origin xyz="0.234 0.0 0.092" rpy="0 0 0"/>
 	</xacro:sensor_orbbec_astra>
-	<!-- Gazebo ros2 control plugins -->
-	<!-- <xacro:ros2_control/> -->
+    <!-- ROS2 Control hardware interface for Gazebo -->
+    <ros2_control name="diff_drive" type="system">
+      <hardware>
+          <plugin>gazebo_ros2_control/GazeboSystem</plugin>
+      </hardware>
+      <joint name="$(arg prefix)left_wheel_joint">
+        <command_interface name="velocity">
+          <param name="min">-1</param>
+          <param name="max">1</param>
+        </command_interface>
+        <state_interface name="position"/>
+        <state_interface name="velocity"/>
+        <state_interface name="effort"/>
+      </joint>
+      <joint name="$(arg prefix)right_wheel_joint">
+        <command_interface name="velocity">
+          <param name="min">-1</param>
+          <param name="max">1</param>
+        </command_interface>
+        <state_interface name="position"/>
+        <state_interface name="velocity"/>
+        <state_interface name="effort"/>
+      </joint>
+    </ros2_control>
+    <!-- Gazebo ROS2 Control Plugin -->
+	<gazebo>
+		<plugin filename="libgazebo_ros2_control.so" name="gazebo_ros2_control">
+            <robot_sim_type>gazebo_ros2_control/GazeboSystem</robot_sim_type>
+            <robot_param_node>/rb1_robot/robot_state_publisher</robot_param_node>
+		    <parameters>$(find rb1_ros2_description)/config/rb1_controller.yaml</parameters>
+		</plugin>
+	</gazebo>
 </robot>

Commit message: Added elevator platform joint

File: xacro/rb1_ros2_base.urdf.xacro (robot description, xacro)
@@ -86,25 +86,34 @@
     <!-- ROS2 Control hardware interface for Gazebo -->
     <ros2_control name="diff_drive" type="system">
-      <hardware>
-          <plugin>gazebo_ros2_control/GazeboSystem</plugin>
-      </hardware>
-      <joint name="$(arg prefix)left_wheel_joint">
-        <command_interface name="velocity">
-          <param name="min">-1</param>
-          <param name="max">1</param>
-        </command_interface>
-        <state_interface name="position"/>
-        <state_interface name="velocity"/>
-        <state_interface name="effort"/>
-      </joint>
-      <joint name="$(arg prefix)right_wheel_joint">
-        <command_interface name="velocity">
-          <param name="min">-1</param>
-          <param name="max">1</param>
-        </command_interface>
-        <state_interface name="position"/>
-        <state_interface name="velocity"/>
-        <state_interface name="effort"/>
-      </joint>
+        <hardware>
+            <plugin>gazebo_ros2_control/GazeboSystem</plugin>
+        </hardware>
+        <joint name="$(arg prefix)left_wheel_joint">
+            <command_interface name="velocity">
+                <param name="min">-1</param>
+                <param name="max">1</param>
+            </command_interface>
+            <state_interface name="position"/>
+            <state_interface name="velocity"/>
+            <state_interface name="effort"/>
+        </joint>
+        <joint name="$(arg prefix)right_wheel_joint">
+            <command_interface name="velocity">
+                <param name="min">-1</param>
+                <param name="max">1</param>
+            </command_interface>
+            <state_interface name="position"/>
+            <state_interface name="velocity"/>
+            <state_interface name="effort"/>
+        </joint>
+        <!-- Elevator joint -->
+	    <joint name="$(arg prefix)elevator_platform_joint">
+	    	<command_interface name="position">
+	    		<param name="min">0.0</param>
+	    		<param name="max">0.3</param>
+	    	</command_interface>
+	    	<state_interface name="position"/>
+	    	<state_interface name="velocity"/>
+	    </joint>
     </ros2_control>
     <!-- Gazebo ROS2 Control Plugin -->
